File: KiCAD/KiCAD_BLEModule/KiCAD_BLEModuleDevTestBoard.sch (KiCad schematic (older format))
At the start: 60 parts, among them J1 PinHeader2.54mm_8, J2 PinHeader2.54mm_2x16, J3 USB-TYPE-C-31-M-17, SW1 SW_Tact_1105, SW10 SW_Tact_1105, SW11 SW_Tact_1105, SW12 SW_Tact_1105, SW13 SW_Tact_1105, SW14 SW_Tact_1105, SW15 SW_Tact_1105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

Commit message: KSG : 거버파일 생성 & 잘못된 다이오드 정보 수정
Parts:
- D1, D10, D11, D12, D13, D14, D15, D16, D2, D3, D4, D5, D6, D7, D8, D9: Shop https://www.devicemart.co.kr/order/cart -> https://www.devicemart.co.kr/goods/view?no=11911
Changed lines of the file:
@@
 F 1 "SS14" H 2000 5634 50  0000 C CNN
 F 2 "digikey-footprints:DO-214AC" H 2150 5700 60  0001 L CNN
-F 3 ".\\Dataseets\\Korean-Hroparts-Elec-TYPE-C-31-M-17.pdf" H 2150 5800 60  0001 L CNN
-F 4 "https://www.devicemart.co.kr/order/cart" H 2150 6400 60  0001 L CNN "Shop"
+F 3 ".\\Dataseets\\SS12~SS110.pdf" H 2150 5800 60  0001 L CNN
+F 4 "https://www.devicemart.co.kr/goods/view?no=11911" H 2150 6400 60  0001 L CNN "Shop"
 F 5 "DIODE SCHOTTKY 40V 1A SMA" H 2150 6500 60  0001 L CNN "Description"
 	1    1950 5500
@@
 F 1 "SS14" H 3100 5634 50  0000 C CNN
 F 2 "digikey-footprints:DO-214AC" H 3250 5700 60  0001 L CNN
-F 3 ".\\Dataseets\\Korean-Hroparts-Elec-TYPE-C-31-M-17.pdf" H 3250 5800 60  0001 L CNN
-F 4 "https://www.devicemart.co.kr/order/cart" H 3250 6400 60  0001 L CNN "Shop"
+F 3 ".\\Dataseets\\SS12~SS110.pdf" H 3250 5800 60  0001 L CNN
+F 4 "https://www.devicemart.co.kr/goods/view?no=11911" H 3250 6400 60  0001 L CNN "Shop"
 F 5 "DIODE SCHOTTKY 40V 1A SMA" H 3250 6500 60  0001 L CNN "Description"
 	1    3050 5500
@@
 F 1 "SS14" H 4200 5634 50  0000 C CNN
 F 2 "digikey-footprints:DO-214AC" H 4350 5700 60  0001 L CNN
-F 3 ".\\Dataseets\\Korean-Hroparts-Elec-TYPE-C-31-M-17.pdf" H 4350 5800 60  0001 L CNN
-F 4 "https://www.devicemart.co.kr/order/cart" H 4350 6400 60  0001 L CNN "Shop"
+F 3 ".\\Dataseets\\SS12~SS110.pdf" H 4350 5800 60  0001 L CNN
+F 4 "https://www.devicemart.co.kr/goods/view?no=11911" H 4350 6400 60  0001 L CNN "Shop"
 F 5 "DIODE SCHOTTKY 40V 1A SMA" H 4350 6500 60  0001 L CNN "Description"
 	1    4150 5500
@@
 F 1 "SS14" H 2000 6234 50  0000 C CNN
 F 2 "digikey-footprints:DO-214AC" H 2150 6300 60  0001 L CNN
-F 3 ".\\Dataseets\\Korean-Hroparts-Elec-TYPE-C-31-M-17.pdf" H 2150 6400 60  0001 L CNN
-F 4 "https://www.devicemart.co.kr/order/cart" H 2150 7000 60  0001 L CNN "Shop"
+F 3 ".\\Dataseets\\SS12~SS110.pdf" H 2150 6400 60  0001 L CNN
+F 4 "https://www.devicemart.co.kr/goods/view?no=11911" H 2150 7000 60  0001 L CNN "Shop"
 F 5 "DIODE SCHOTTKY 40V 1A SMA" H 2150 7100 60  0001 L CNN "Description"
 	1    1950 6100
@@
 F 1 "SS14" H 3100 6234 50  0000 C CNN
 F 2 "digikey-footprints:DO-214AC" H 3250 6300 60  0001 L CNN
-F 3 ".\\Dataseets\\Korean-Hroparts-Elec-TYPE-C-31-M-17.pdf" H 3250 6400 60  0001 L CNN
-F 4 "https://www.devicemart.co.kr/order/cart" H 3250 7000 60  0001 L CNN "Shop"
+F 3 ".\\Dataseets\\SS12~SS110.pdf" H 3250 6400 60  0001 L CNN
+F 4 "https://www.devicemart.co.kr/goods/view?no=11911" H 3250 7000 60  0001 L CNN "Shop"
 F 5 "DIODE SCHOTTKY 40V 1A SMA" H 3250 7100 60  0001 L CNN "Description"
 	1    3050 6100
@@
 F 1 "SS14" H 4200 6234 50  0000 C CNN
 F 2 "digikey-footprints:DO-214AC" H 4350 6300 60  0001 L CNN
-F 3 ".\\Dataseets\\Korean-Hroparts-Elec-TYPE-C-31-M-17.pdf" H 4350 6400 60  0001 L CNN
-F 4 "https://www.devicemart.co.kr/order/cart" H 4350 7000 60  0001 L CNN "Shop"
+F 3 ".\\Dataseets\\SS12~SS110.pdf" H 4350 6400 60  0001 L CNN
+F 4 "https://www.devicemart.co.kr/goods/view?no=11911" H 4350 7000 60  0001 L CNN "Shop"
 F 5 "DIODE SCHOTTKY 40V 1A SMA" H 4350 7100 60  0001 L CNN "Description"
 	1    4150 6100
@@
 F 1 "SS14" H 2000 6834 50  0000 C CNN
 F 2 "digikey-footprints:DO-214AC" H 2150 6900 60  0001 L CNN
-F 3 ".\\Dataseets\\Korean-Hroparts-Elec-TYPE-C-31-M-17.pdf" H 2150 7000 60  0001 L CNN
-F 4 "https://www.devicemart.co.kr/order/cart" H 2150 7600 60  0001 L CNN "Shop"
+F 3 ".\\Dataseets\\SS12~SS110.pdf" H 2150 7000 60  0001 L CNN
+F 4 "https://www.devicemart.co.kr/goods/view?no=11911" H 2150 7600 60  0001 L CNN "Shop"
 F 5 "DIODE SCHOTTKY 40V 1A SMA" H 2150 7700 60  0001 L CNN "Description"
 	1    1950 6700
@@
 F 1 "SS14" H 3100 6834 50  0000 C CNN
 F 2 "digikey-footprints:DO-214AC" H 3250 6900 60  0001 L CNN
-F 3 ".\\Dataseets\\Korean-Hroparts-Elec-TYPE-C-31-M-17.pdf" H 3250 7000 60  0001 L CNN
-F 4 "https://www.devicemart.co.kr/order/cart" H 3250 7600 60  0001 L CNN "Shop"
+F 3 ".\\Dataseets\\SS12~SS110.pdf" H 3250 7000 60  0001 L CNN
+F 4 "https://www.devicemart.co.kr/goods/view?no=11911" H 3250 7600 60  0001 L CNN "Shop"
 F 5 "DIODE SCHOTTKY 40V 1A SMA" H 3250 7700 60  0001 L CNN "Description"
 	1    3050 6700
@@
 F 1 "SS14" H 4200 6834 50  0000 C CNN
 F 2 "digikey-footprints:DO-214AC" H 4350 6900 60  0001 L CNN
-F 3 ".\\Dataseets\\Korean-Hroparts-Elec-TYPE-C-31-M-17.pdf" H 4350 7000 60  0001 L CNN
-F 4 "https://www.devicemart.co.kr/order/cart" H 4350 7600 60  0001 L CNN "Shop"
+F 3 ".\\Dataseets\\SS12~SS110.pdf" H 4350 7000 60  0001 L CNN
+F 4 "https://www.devicemart.co.kr/goods/view?no=11911" H 4350 7600 60  0001 L CNN "Shop"
 F 5 "DIODE SCHOTTKY 40V 1A SMA" H 4350 7700 60  0001 L CNN "Description"
 	1    4150 6700
@@
 F 1 "SS14" H 2000 7434 50  0000 C CNN
 F 2 "digikey-footprints:DO-214AC" H 2150 7500 60  0001 L CNN
-F 3 ".\\Dataseets\\Korean-Hroparts-Elec-TYPE-C-31-M-17.pdf" H 2150 7600 60  0001 L CNN
-F 4 "https://www.devicemart.co.kr/order/cart" H 2150 8200 60  0001 L CNN "Shop"
+F 3 ".\\Dataseets\\SS12~SS110.pdf" H 2150 7600 60  0001 L CNN
+F 4 "https://www.devicemart.co.kr/goods/view?no=11911" H 2150 8200 60  0001 L CNN "Shop"
 F 5 "DIODE SCHOTTKY 40V 1A SMA" H 2150 8300 60  0001 L CNN "Description"
 	1    1950 7300
@@
 F 1 "SS14" H 3100 7434 50  0000 C CNN
 F 2 "digikey-footprints:DO-214AC" H 3250 7500 60  0001 L CNN
-F 3 ".\\Dataseets\\Korean-Hroparts-Elec-TYPE-C-31-M-17.pdf" H 3250 7600 60  0001 L CNN
-F 4 "https://www.devicemart.co.kr/order/cart" H 3250 8200 60  0001 L CNN "Shop"
+F 3 ".\\Dataseets\\SS12~SS110.pdf" H 3250 7600 60  0001 L CNN
+F 4 "https://www.devicemart.co.kr/goods/view?no=11911" H 3250 8200 60  0001 L CNN "Shop"
 F 5 "DIODE SCHOTTKY 40V 1A SMA" H 3250 8300 60  0001 L CNN "Description"
 	1    3050 7300
@@
 F 1 "SS14" H 4200 7434 50  0000 C CNN
 F 2 "digikey-footprints:DO-214AC" H 4350 7500 60  0001 L CNN
-F 3 ".\\Dataseets\\Korean-Hroparts-Elec-TYPE-C-31-M-17.pdf" H 4350 7600 60  0001 L CNN
-F 4 "https://www.devicemart.co.kr/order/cart" H 4350 8200 60  0001 L CNN "Shop"
+F 3 ".\\Dataseets\\SS12~SS110.pdf" H 4350 7600 60  0001 L CNN
+F 4 "https://www.devicemart.co.kr/goods/view?no=11911" H 4350 8200 60  0001 L CNN "Shop"
 F 5 "DIODE SCHOTTKY 40V 1A SMA" H 4350 8300 60  0001 L CNN "Description"
 	1    4150 7300
@@
 F 1 "SS14" H 5300 5634 50  0000 C CNN
 F 2 "digikey-footprints:DO-214AC" H 5450 5700 60  0001 L CNN
-F 3 ".\\Dataseets\\Korean-Hroparts-Elec-TYPE-C-31-M-17.pdf" H 5450 5800 60  0001 L CNN
-F 4 "https://www.devicemart.co.kr/order/cart" H 5450 6400 60  0001 L CNN "Shop"
+F 3 ".\\Dataseets\\SS12~SS110.pdf" H 5450 5800 60  0001 L CNN
+F 4 "https://www.devicemart.co.kr/goods/view?no=11911" H 5450 6400 60  0001 L CNN "Shop"
 F 5 "DIODE SCHOTTKY 40V 1A SMA" H 5450 6500 60  0001 L CNN "Description"
 	1    5250 5500
@@
 F 1 "SS14" H 5300 6234 50  0000 C CNN
 F 2 "digikey-footprints:DO-214AC" H 5450 6300 60  0001 L CNN
-F 3 ".\\Dataseets\\Korean-Hroparts-Elec-TYPE-C-31-M-17.pdf" H 5450 6400 60  0001 L CNN
-F 4 "https://www.devicemart.co.kr/order/cart" H 5450 7000 60  0001 L CNN "Shop"
+F 3 ".\\Dataseets\\SS12~SS110.pdf" H 5450 6400 60  0001 L CNN
+F 4 "https://www.devicemart.co.kr/goods/view?no=11911" H 5450 7000 60  0001 L CNN "Shop"
 F 5 "DIODE SCHOTTKY 40V 1A SMA" H 5450 7100 60  0001 L CNN "Description"
 	1    5250 6100
@@
 F 1 "SS14" H 5300 6834 50  0000 C CNN
 F 2 "digikey-footprints:DO-214AC" H 5450 6900 60  0001 L CNN
-F 3 ".\\Dataseets\\Korean-Hroparts-Elec-TYPE-C-31-M-17.pdf" H 5450 7000 60  0001 L CNN
-F 4 "https://www.devicemart.co.kr/order/cart" H 5450 7600 60  0001 L CNN "Shop"
+F 3 ".\\Dataseets\\SS12~SS110.pdf" H 5450 7000 60  0001 L CNN
+F 4 "https://www.devicemart.co.kr/goods/view?no=11911" H 5450 7600 60  0001 L CNN "Shop"
 F 5 "DIODE SCHOTTKY 40V 1A SMA" H 5450 7700 60  0001 L CNN "Description"
 	1    5250 6700
@@
 F 1 "SS14" H 5300 7434 50  0000 C CNN
 F 2 "digikey-footprints:DO-214AC" H 5450 7500 60  0001 L CNN
-F 3 ".\\Dataseets\\Korean-Hroparts-Elec-TYPE-C-31-M-17.pdf" H 5450 7600 60  0001 L CNN
-F 4 "https://www.devicemart.co.kr/order/cart" H 5450 8200 60  0001 L CNN "Shop"
+F 3 ".\\Dataseets\\SS12~SS110.pdf" H 5450 7600 60  0001 L CNN
+F 4 "https://www.devicemart.co.kr/goods/view?no=11911" H 5450 8200 60  0001 L CNN "Shop"
 F 5 "DIODE SCHOTTKY 40V 1A SMA" H 5450 8300 60  0001 L CNN "Description"
 	1    5250 7300
